File: DRSSTC High Power Distribution Board/DRSSTC High Power Distribution Board.kicad_pcb (KiCad board)
At the start: 2 copper layers, 100 x 56.8 mm, 8 parts, among them U1 KF635-6.35-2P, U2 KF635-6.35-2P, U3 FC-DLSF2515-1.0MH/30A-L, U4 KF950-9.5-3P

Commit message: Initial commit of components
Parts:
- C1, C2: footprint Custom Parts:CAP-TH_L13.0-W6.0-P10.00-D0.6 -> parts:CAP-TH_L13.0-W6.0-P10.00-D0.6
- C3: footprint Custom Parts:CAP-TH_L26.5-W11.0-P22.50-D1.4 -> parts:CAP-TH_L26.5-W11.0-P22.50-D1.4
- D1: footprint Custom Parts:TO-247-3_L15.9-W5.1-P5.44-L -> parts:TO-247-3_L15.9-W5.1-P5.44-L
- U1, U2: footprint Custom Parts:CONN-TH_P6.35_KF635-6.35-2P -> parts:CONN-TH_P6.35_KF635-6.35-2P
- U3: footprint Custom Parts:FILTER-TH_8P-L25.0-W18.0 -> parts:FILTER-TH_8P-L25.0-W18.0
- U4: footprint Custom Parts:CONN-TH_3P-P9.50_KF950-9.5-3P -> easyeda2kicad:CONN-TH_3P-P9.50_KF950-9.5-3P
Changed lines of the file:
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@@
 	(net 6 "E")
 	(net 7 "N")
-	(footprint "Custom Parts:FILTER-TH_8P-L25.0-W18.0"
+	(footprint "parts:FILTER-TH_8P-L25.0-W18.0"
 		(layer "F.Cu")
 		(at 175 73.5 90)
@@
 		)
 		(embedded_fonts no)
-		(model "${EASYEDA2KICAD}/easyeda2kicad.3dshapes/FILTER-TH_8P-L25.0-W18.0.wrl"
+		(model "${KIPRJMOD}/Custom Parts/parts.3dmodels/FILTER-TH_8P-L25.0-W18.0.step"
 			(offset
 				(xyz -0 -0 14)
@@
 		)
 	)
-	(footprint "Custom Parts:CONN-TH_P6.35_KF635-6.35-2P"
+	(footprint "parts:CONN-TH_P6.35_KF635-6.35-2P"
 		(layer "F.Cu")
 		(at 209.5 52.5 180)
@@
 		)
 		(embedded_fonts no)
-		(model "${EASYEDA2KICAD}/easyeda2kicad.3dshapes/CONN-TH_P6.35_KF635-6.35-2P.wrl"
+		(model "${KIPRJMOD}/Custom Parts/parts.3dmodels/CONN-TH_P6.35_KF635-6.35-2P.step"
 			(offset
 				(xyz -0.2 -0.8 0)
@@
 		)
 	)
-	(footprint "Custom Parts:CONN-TH_P6.35_KF635-6.35-2P"
+	(footprint "parts:CONN-TH_P6.35_KF635-6.35-2P"
 		(layer "F.Cu")
 		(at 137.75 73.545 -90)
@@
 		)
 		(embedded_fonts no)
-		(model "${EASYEDA2KICAD}/easyeda2kicad.3dshapes/CONN-TH_P6.35_KF635-6.35-2P.wrl"
+		(model "${KIPRJMOD}/Custom Parts/parts.3dmodels/CONN-TH_P6.35_KF635-6.35-2P.step"
 			(offset
 				(xyz -0.2 -0.8 0)
@@
 		)
 	)
-	(footprint "Custom Parts:CONN-TH_3P-P9.50_KF950-9.5-3P"
+	(footprint "easyeda2kicad:CONN-TH_3P-P9.50_KF950-9.5-3P"
 		(layer "F.Cu")
 		(at 222.75 73.6175 90)
@@
 			(at 0 4 90)
 			(layer "F.Fab")
-			(hide yes)
 			(effects
 				(font
@@
 		(sheetname "/")
 		(sheetfile "DRSSTC High Power Distribution Board.kicad_sch")
-		(zone_connect 2)
 		(attr through_hole)
 		(fp_line
@@
 		)
 	)
-	(footprint "Custom Parts:CAP-TH_L13.0-W6.0-P10.00-D0.6"
+	(footprint "parts:CAP-TH_L13.0-W6.0-P10.00-D0.6"
 		(layer "F.Cu")
 		(at 190.67 56 90)
@@
 		)
 		(embedded_fonts no)
-		(model "${EASYEDA2KICAD}/easyeda2kicad.3dshapes/CAP-TH_L13.0-W6.0-H12.0-P10.0.wrl"
+		(model "${KIPRJMOD}/Custom Parts/parts.3dmodels/CAP-TH_L13.0-W6.0-H12.0-P10.0.step"
 			(offset
 				(xyz 0 -3 6)
@@
 		)
 	)
-	(footprint "Custom Parts:CAP-TH_L26.5-W11.0-P22.50-D1.4"
+	(footprint "parts:CAP-TH_L26.5-W11.0-P22.50-D1.4"
 		(layer "F.Cu")
 		(at 154.5 73.6 90)
@@
 		)
 		(embedded_fonts no)
-		(model "${EASYEDA2KICAD}/easyeda2kicad.3dshapes/CAP-TH_L26.5-W11.0-H23.0-P22.5.wrl"
+		(model "${KIPRJMOD}/Custom Parts/parts.3dmodels/CAP-TH_L26.5-W11.0-H23.0-P22.5.step"
 			(offset
 				(xyz 0 -5.5 11.5)
@@
 		)
 	)
-	(footprint "Custom Parts:TO-247-3_L15.9-W5.1-P5.44-L"
+	(footprint "parts:TO-247-3_L15.9-W5.1-P5.44-L"
 		(layer "F.Cu")
 		(at 192.81 99 180)
@@
 		)
 		(embedded_fonts no)
-		(model "${EASYEDA2KICAD}/easyeda2kicad.3dshapes/TO-247_3PIN-L15.9-W5.1-H25.0-P5.44-L.wrl"
+		(model "${KICAD9_3DMODEL_DIR}/Package_TO_SOT_THT.3dshapes/TO-247-3_Vertical.step"
 			(offset
-				(xyz 0 0.3 11)
+				(xyz -5.5 0 0)
 			)
 			(scale
@@
 			)
 			(rotate
-				(xyz 0 0 0)
+				(xyz -0 -0 -0)
 			)
 		)
 	)
-	(footprint "Custom Parts:CAP-TH_L13.0-W6.0-P10.00-D0.6"
+	(footprint "parts:CAP-TH_L13.0-W6.0-P10.00-D0.6"
 		(layer "F.Cu")
 		(at 198.17 56 -90)
@@
 		)
 		(embedded_fonts no)
-		(model "${EASYEDA2KICAD}/easyeda2kicad.3dshapes/CAP-TH_L13.0-W6.0-H12.0-P10.0.wrl"
+		(model "${KIPRJMOD}/Custom Parts/parts.3dmodels/CAP-TH_L13.0-W6.0-H12.0-P10.0.step"
 			(offset
 				(xyz 0 -3 6)
