File: DRSSTC High Power Distribution Board/DRSSTC High Power Distribution Board.kicad_sch (KiCad schematic)
At the start: 8 parts, among them U1 KF635-6.35-2P, U2 KF635-6.35-2P, U3 FC-DLSF2515-1.0MH/30A-L, U4 KF950-9.5-3P

Commit message: Initial commit of components
Parts:
- C1, C2: footprint Custom Parts:CAP-TH_L13.0-W6.0-P10.00-D0.6 -> parts:CAP-TH_L13.0-W6.0-P10.00-D0.6; symbol Custom Parts:C_Small -> parts:C_Small
- C3: footprint Custom Parts:CAP-TH_L26.5-W11.0-P22.50-D1.4 -> parts:CAP-TH_L26.5-W11.0-P22.50-D1.4; symbol Custom Parts:C_Small -> parts:C_Small
- D1: footprint Custom Parts:TO-247-3_L15.9-W5.1-P5.44-L -> parts:TO-247-3_L15.9-W5.1-P5.44-L; symbol Custom Parts:DSP45-16A -> parts:DSP45-16A
- U1, U2: footprint Custom Parts:CONN-TH_P6.35_KF635-6.35-2P -> parts:CONN-TH_P6.35_KF635-6.35-2P; symbol Custom Parts:KF635-6.35-2P -> parts:KF635-6.35-2P
- U3: footprint Custom Parts:FILTER-TH_8P-L25.0-W18.0 -> parts:FILTER-TH_8P-L25.0-W18.0; symbol Custom Parts:FC-DLSF2515-1.0MH_30A-L -> parts:FC-DLSF2515-1.0MH_30A-L
- U4: footprint Custom Parts:CONN-TH_3P-P9.50_KF950-9.5-3P -> easyeda2kicad:CONN-TH_3P-P9.50_KF950-9.5-3P; symbol Custom Parts:KF950-9.5-3P -> parts:KF950-9.5-3P
Changed lines of the file:
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@@
 	)
 	(symbol
-		(lib_id "Custom Parts:C_Small")
+		(lib_id "parts:C_Small")
 		(at 115.57 63.5 0)
 		(unit 1)
@@
 			)
 		)
-		(property "Footprint" "Custom Parts:CAP-TH_L26.5-W11.0-P22.50-D1.4"
+		(property "Footprint" "parts:CAP-TH_L26.5-W11.0-P22.50-D1.4"
 			(at 115.57 63.5 0)
 			(effects
@@
 	)
 	(symbol
-		(lib_id "Custom Parts:KF950-9.5-3P")
+		(lib_id "parts:KF950-9.5-3P")
 		(at 182.88 59.69 0)
 		(mirror x)
@@
 			)
 		)
-		(property "Footprint" "Custom Parts:CONN-TH_3P-P9.50_KF950-9.5-3P"
+		(property "Footprint" "easyeda2kicad:CONN-TH_3P-P9.50_KF950-9.5-3P"
 			(at 182.88 49.53 0)
 			(effects
@@
 	)
 	(symbol
-		(lib_id "Custom Parts:FC-DLSF2515-1.0MH_30A-L")
+		(lib_id "parts:FC-DLSF2515-1.0MH_30A-L")
 		(at 128.27 63.5 90)
 		(mirror x)
@@
 			)
 		)
-		(property "Footprint" "Custom Parts:FILTER-TH_8P-L25.0-W18.0"
+		(property "Footprint" "parts:FILTER-TH_8P-L25.0-W18.0"
 			(at 139.7 63.5 0)
 			(effects
@@
 	)
 	(symbol
-		(lib_id "Custom Parts:KF635-6.35-2P")
+		(lib_id "parts:KF635-6.35-2P")
 		(at 95.25 59.69 180)
 		(unit 1)
@@
 			)
 		)
-		(property "Footprint" "Custom Parts:CONN-TH_P6.35_KF635-6.35-2P"
+		(property "Footprint" "parts:CONN-TH_P6.35_KF635-6.35-2P"
 			(at 95.25 50.8 0)
 			(effects
@@
 	)
 	(symbol
-		(lib_id "Custom Parts:KF635-6.35-2P")
+		(lib_id "parts:KF635-6.35-2P")
 		(at 90.17 76.2 180)
 		(unit 1)
@@
 			)
 		)
-		(property "Footprint" "Custom Parts:CONN-TH_P6.35_KF635-6.35-2P"
+		(property "Footprint" "parts:CONN-TH_P6.35_KF635-6.35-2P"
 			(at 90.17 67.31 0)
 			(effects
@@
 	)
 	(symbol
-		(lib_id "Custom Parts:DSP45-16A")
+		(lib_id "parts:DSP45-16A")
 		(at 160.02 58.42 0)
 		(unit 1)
@@
 			)
 		)
-		(property "Footprint" "Custom Parts:TO-247-3_L15.9-W5.1-P5.44-L"
+		(property "Footprint" "parts:TO-247-3_L15.9-W5.1-P5.44-L"
 			(at 160.02 68.58 0)
 			(effects
@@
 	)
 	(symbol
-		(lib_id "Custom Parts:C_Small")
+		(lib_id "parts:C_Small")
 		(at 140.97 57.15 0)
 		(unit 1)
@@
 			)
 		)
-		(property "Footprint" "Custom Parts:CAP-TH_L13.0-W6.0-P10.00-D0.6"
+		(property "Footprint" "parts:CAP-TH_L13.0-W6.0-P10.00-D0.6"
 			(at 140.97 57.15 0)
 			(effects
@@
 	)
 	(symbol
-		(lib_id "Custom Parts:C_Small")
+		(lib_id "parts:C_Small")
 		(at 140.97 64.77 0)
 		(unit 1)
@@
 			)
 		)
-		(property "Footprint" "Custom Parts:CAP-TH_L13.0-W6.0-P10.00-D0.6"
+		(property "Footprint" "parts:CAP-TH_L13.0-W6.0-P10.00-D0.6"
 			(at 140.97 64.77 0)
 			(effects
