File: DRSSTC MIDI Interrupter 2/DRSSTC MIDI Interrupter 2.kicad_pcb (KiCad board)
At the start: 2 copper layers, 63 parts, among them CN2 HX25003-2WAP, Q1 8205A_C5370944, Q2 AO3401A_C347476, U1 ESP32-S3-WROOM-1, U10 TPS63802DLAR, U11 BQ27441DRZR-G1B, U2 BQ24072RGT, U3 DW01A, U4 TPS61023DRLR, U6 SRV05-4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

Commit message: Initial commit of components
Parts:
- added J1: ~, parts:LCD, F.Cu at (194.5, 74.6)
- added R28: 10kΩ, Resistor_SMD:R_0805_2012Metric_Pad1.20x1.40mm_HandSolder, F.Cu at (146.4, 129.5)
- added R29: 10kΩ, Resistor_SMD:R_0805_2012Metric_Pad1.20x1.40mm_HandSolder, F.Cu at (146.4, 132.5)
- added U5: RP2040, Package_DFN_QFN:QFN-56-1EP_7x7mm_P0.4mm_EP3.2x3.2mm, F.Cu at (171.2, 130.7)
- moved U7 48.5 mm to (175.2, 101.9)
- moved U8 47.6 mm to (156.4, 133.2)
- moved R7 44.6 mm to (151.7, 133.4)
- moved U2 42.2 mm to (167.4, 109.0)
- moved Q2 42.0 mm to (166.5, 113.8)
- moved Q1 41.5 mm to (171.9, 76.2)
- moved U6 41.5 mm to (171.9, 80.8)
- moved U3 41.5 mm to (166.9, 76.4)
- moved U9 41.5 mm to (166.9, 81.0)
- moved U4 41.5 mm to (159.6, 133.1)
- moved U11 40.6 mm to (166.6, 103.0)
- moved R10 40.3 mm to (171.0, 101.6)
- moved R11 40.3 mm to (171.0, 104.5)
- moved U10 35.2 mm to (172.1, 113.9)
- moved L3 35.2 mm to (168.9, 96.2)
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Connections:
- U1 pad 16: unconnected-(U1-IO46-Pad16) -> AVOID_FOR_NOW_ONLY_INPUT
- U1 pad 17: unconnected-(U1-IO9-Pad17) -> TOUCH_IRQ
- U1 pad 18: unconnected-(U1-IO10-Pad18) -> TOUCH_MOSI
- U1 pad 19: unconnected-(U1-IO11-Pad19) -> TOUCH_CS
- U1 pad 20: unconnected-(U1-IO12-Pad20) -> TOUCH_CLK
- U1 pad 21: unconnected-(U1-IO13-Pad21) -> LCD_RS
- U1 pad 22: unconnected-(U1-IO14-Pad22) -> LCD_RD
- U1 pad 23: unconnected-(U1-IO21-Pad23) -> LCD_LED_A
- U1 pad 24: unconnected-(U1-IO47-Pad24) -> LCD_CS
- U1 pad 25: unconnected-(U1-IO48-Pad25) -> LCD_WR
- U1 pad 26: unconnected-(U1-IO45-Pad26) -> LCD_DB0
- U1 pad 31: unconnected-(U1-IO38-Pad31) -> LCD_DB1
- U1 pad 32: unconnected-(U1-IO39-Pad32) -> LCD_DB2
- U1 pad 33: unconnected-(U1-IO40-Pad33) -> LCD_DB3
- U1 pad 34: unconnected-(U1-IO41-Pad34) -> LCD_DB4
- U1 pad 35: unconnected-(U1-IO42-Pad35) -> LCD_DB5
- U1 pad 38: unconnected-(U1-IO2-Pad38) -> LCD_DB6
- U1 pad 39: unconnected-(U1-IO1-Pad39) -> LCD_DB7
- U1 pad 8: unconnected-(U1-IO15-Pad8) -> TOUCH_MISO
- U1 pad 9: unconnected-(U1-IO16-Pad9) -> LCD_RESET
